Commit message: Lynx: make fixed base_footprint optional (ROBOT_PUBLISH_BASE_FOOTPRINT)
New env var ROBOT_PUBLISH_BASE_FOOTPRINT (default true = unchanged upstream
URDF) is passed to the Lynx xacro as publish_base_footprint. With false, the
fixed body_link -> base_footprint joint and the base_footprint link are omitted,
so a localization can publish base_footprint as a gravity-aligned frame
(odom -> base_footprint -> base_link, REP-120) without a second parent.

Co-Authored-By: Claude Opus 5.5 <noreply@anthropic.com>
Claude-Session: https://claude.ai/code/session_01RWFZfkDLVjvURCSGbyVRSs

File: husarion_ugv_description/urdf/lynx.urdf.xacro (robot description, xacro)
@@ -11,4 +11,5 @@
     default="" />
   <xacro:arg name="namespace" default="" />
+  <xacro:arg name="publish_base_footprint" default="true" />
   <xacro:include filename="$(find husarion_ugv_description)/urdf/lynx/lynx_macro.urdf.xacro" ns="husarion" />
   <xacro:husarion.lynx_robot
@@ -19,5 +20,6 @@
     controller_config_file="$(arg controller_config_file)"
     battery_config_file="$(arg battery_config_file)"
-    namespace="$(arg namespace)" />
+    namespace="$(arg namespace)"
+    publish_base_footprint="$(arg publish_base_footprint)" />
   <xacro:arg name="components_config_path" default="$(find husarion_ugv_description)/config/components.yaml" />
   <xacro:property name="components_config_path_property" value="$(arg components_config_path)" />

File: husarion_ugv_description/urdf/lynx/base.urdf.xacro (robot description, xacro)
@@ -3,5 +3,5 @@
   <xacro:macro
     name="body"
-    params="wheel_radius imu_xyz imu_rpy">
+    params="wheel_radius imu_xyz imu_rpy publish_base_footprint:=true">
     <joint name="base_to_body_joint" type="fixed">
       <origin xyz="0.0 0.0 0.0" rpy="0.0 0.0 0.0" />
@@ -30,10 +30,14 @@
       </inertial>
     </link>
-    <joint name="body_to_footprint_joint" type="fixed">
-      <origin xyz="0.0 0.0 -${wheel_radius}" rpy="0.0 0.0 0.0" />
-      <parent link="body_link" />
-      <child link="base_footprint" />
-    </joint>
-    <link name="base_footprint" />
+    <!-- Disable when base_footprint is published as a gravity-aligned (planar) frame by the localization,
+         e.g. odom -> base_footprint -> base_link (REP-120). A fixed joint here would give it a second parent. -->
+    <xacro:if value="${publish_base_footprint}">
+      <joint name="body_to_footprint_joint" type="fixed">
+        <origin xyz="0.0 0.0 -${wheel_radius}" rpy="0.0 0.0 0.0" />
+        <parent link="body_link" />
+        <child link="base_footprint" />
+      </joint>
+      <link name="base_footprint" />
+    </xacro:if>
     <joint name="body_to_imu_joint" type="fixed">
       <origin xyz="${imu_xyz}" rpy="${imu_rpy}" />

File: husarion_ugv_description/urdf/lynx/lynx_macro.urdf.xacro (robot description, xacro)
@@ -10,5 +10,6 @@
             imu_rpy:='0.0 0.0 -1.57'
             namespace:=''
-            use_madgwick_filter:=false">
+            use_madgwick_filter:=false
+            publish_base_footprint:=true">
     <xacro:if value="${use_sim}">
       <xacro:property name="imu_xyz" value="0.052 0.073 -0.006" />
@@ -27,5 +28,6 @@
       wheel_radius="${wheel_config['wheel_radius']}"
       imu_xyz="${imu_xyz}"
-      imu_rpy="${imu_rpy}" />
+      imu_rpy="${imu_rpy}"
+      publish_base_footprint="${publish_base_footprint}" />
     <!-- WHEEL DECLARATION -->
     <xacro:wheel.wheel
